File: tiny-12V-programmer/tiny-12V-programmer.kicad_pcb (KiCad board)
At the start: 2 copper layers, 60 x 60 mm, 25 parts, among them J1 Conn_01x02_Female, J10 GND, J2 Conn_01x02_Female, J3 PB0, J4 ISP, J5 PB1, J6 PB2, J7 PB3, J8 Conn_01x03_Female, J9 VCC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

Commit message: v1
Routing:
- net Net-(SW2-Pad2): track 57.3 -> 34.1 mm
- net Net-(SW2-Pad5): track 49.0 -> 57.4 mm
- net Net-(Q1-Pad2): track 29.5 -> 31.9 mm
- net Net-(SW2-Pad8): track 45.2 -> 46.8 mm
- net +12V: track 49.0 -> 50.3 mm
- net Net-(J5-Pad1): track 59.1 -> 60.2 mm
- net Net-(J7-Pad1): track 33.5 -> 34.5 mm
Other:
- board text added: "ATTiny10 12V programmer"
- board text added: "kaleidoscope 2020 v1"
- board text added: "program"
- board text added: "run"

Commit message: Corrections to v1
Parts:
- moved U2 0.38 mm to (76.5, 83.5)
Routing:
- net Net-(SW2-Pad5): track 57.4 -> 59.0 mm
- net Net-(SW2-Pad8): track 46.8 -> 45.2 mm
- net Net-(J6-Pad1): track 38.7 -> 37.9 mm
Other:
- board text added: "12V"
- board text added: "5V"
- board text added: "GND"
- board text added: "kaleidoscope 2020 v2"
- board text removed: "kaleidoscope 2020 v1"
