File: tiny-12V-programmer/tiny-12V-programmer.sch (KiCad schematic (older format))
At the start: 22 parts, among them J1 Conn_01x02_Female, J10 GND, J2 Conn_01x02_Female, J3 PB0, J4 ISP, J5 PB1, J6 PB2, J7 PB3, J8 Conn_01x03_Female, J9 VCC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

Commit message: Corrections to v1
Other:
- note added: "TODO: smaller PNP\nTODO: 5V regulator\nTODO: LED for programming"
Changed lines of the file:
@@
 Wire Wire Line
 	3750 5350 3750 5550
+Text Notes 8250 1950 0    50   ~ 0
+TODO: smaller PNP\nTODO: 5V regulator\nTODO: LED for programming
 $EndSCHEMATC

Commit message: Blinky for attiny10
Other:
- note added: "TODO: smaller PNP\nTODO: 5V regulator\nTODO: LED for programming\nTODO: turn TPI connector (J4) 180"
- note removed: "TODO: smaller PNP\nTODO: 5V regulator\nTODO: LED for programming"
Changed lines of the file:
@@
 	3750 5350 3750 5550
 Text Notes 8250 1950 0    50   ~ 0
-TODO: smaller PNP\nTODO: 5V regulator\nTODO: LED for programming
+TODO: smaller PNP\nTODO: 5V regulator\nTODO: LED for programming\nTODO: turn TPI connector (J4) 180
 $EndSCHEMATC
